Commit message: added apriltag texture model

File: catkin_ws/src/auefinals/aue_finals/urdf/aprilTag_robot/common_properties.xacro (robot description, xacro)
@@ -1,4 +1,4 @@
 <?xml version="1.0" ?>
-<robot name="xacro_properties" xmlns:xacro="http://ros.org/wiki/xacro">
+<robot name="xacro_properties2" xmlns:xacro="http://ros.org/wiki/xacro">
   <!-- Init colour -->
   <material name="black">
@@ -10,4 +10,7 @@
   <material name="light_black">
     <color rgba="0.4 0.4 0.4 1.0"/>
+  </material>
+  <material name="aprilTag">
+    <color rgba="0.1 0.0 0.0 1.0"/>
   </material>
   <material name="blue">

File: catkin_ws/src/auefinals/aue_finals/urdf/aprilTag_robot/turtlebot3_burger.gazebo.xacro (robot description, xacro)
@@ -1,8 +1,19 @@
 <?xml version="1.0"?>
-<robot name="turtlebot3_burger_sim" xmlns:xacro="http://ros.org/wiki/xacro">
+<robot name="turtlebot3_2_sim" xmlns:xacro="http://ros.org/wiki/xacro">
+  <!--env name="GAZEBO_MODEL_PATH" value="$(find aue_finals)/models"/-->
   <xacro:arg name="laser_visual" default="false"/>
   <xacro:arg name="imu_visual"   default="false"/>
   <gazebo reference="base_link">
     <material>Gazebo/DarkGrey</material>
+  </gazebo>
+  <gazebo reference="aprilTag_link">
+    <!--material>
+      <script>
+         <uri>model://aprilTag/materials/scripts</uri>
+         <uri>model://aprilTag/materials/textures</uri>
+         <name>aprilTag</name>
+      </script>
+    </material-->
+    <material>aprilTag</material>
   </gazebo>
   <gazebo reference="wheel_left_link">

File: catkin_ws/src/auefinals/aue_finals/urdf/aprilTag_robot/turtlebot3_burger.urdf.xacro (robot description, xacro)
@@ -1,6 +1,6 @@
 <?xml version="1.0" ?>
-<robot name="turtlebot3_burger" xmlns:xacro="http://ros.org/wiki/xacro">
-  <xacro:include filename="$(find finalProject)/urdf/original/common_properties.xacro"/>
-  <xacro:include filename="$(find finalProject)/urdf/original/turtlebot3_burger.gazebo.xacro"/>
+<robot name="turtlebot3_2" xmlns:xacro="http://ros.org/wiki/xacro">
+  <xacro:include filename="$(find aue_finals)/urdf/aprilTag_robot/common_properties.xacro"/>
+  <xacro:include filename="$(find aue_finals)/urdf/aprilTag_robot/turtlebot3_burger.gazebo.xacro"/>
   <link name="base_footprint"/>
   <joint name="base_joint" type="fixed">
@@ -30,4 +30,47 @@
                izz="2.0064271e-03" />
     </inertial>
+  </link>
+  <joint name="aprilTag_joint" type="fixed">
+    <parent link="base_link"/>
+    <child link="aprilTag_link"/>
+    <origin xyz=".15 0 0.2" rpy="0 0 0"/>
+  </joint>
+  <link name="aprilTag_link">
+    <visual>
+      <origin xyz="0 0 0" rpy="0 0 0"/>
+      <geometry>
+        <box size="0.05 0.3 0.3"/>
+      </geometry>
+      <!--material>
+        <script>
+          <uri>model://aprilTag/materials/scripts</uri>
+          <uri>model://aprilTag/materials/textures</uri>
+          <name>aprilTag</name>
+        </script>
+      </material-->
+      <!--material name="black"/-->
+    </visual>
+    <collision>
+      <origin xyz="0 0.001 0" rpy="0 0 0"/>
+      <geometry>
+        <box size="0.05 0.3 0.3"/>
+      </geometry>
+    </collision>
+    <inertial>
+      <origin xyz="0 0 0" />
+      <mass value="0.005" />
+      <inertia ixx="0.001" ixy="0.0" ixz="0.0"
+               iyy="0.001" iyz="0.0"
+               izz="0.001" />
+    </inertial>
+    <!--gazebo>
+      <material>
+        <script>
+          <uri>model://aprilTag/materials/scripts</uri>
+          <uri>model://aprilTag/materials/textures</uri>
+          <name>aprilTag</name>
+        </script>
+      </material>
+    </gazebo-->
   </link>
   <joint name="wheel_left_joint" type="continuous">
@@ -140,28 +183,3 @@
     </inertial>
   </link>
-  <joint name="camera_joint" type="fixed">
-    <origin xyz="0.073 -0.011 0.084" rpy="0 0 0"/>
-    <parent link="base_link"/>
-    <child link="camera_link"/>
-  </joint>
-  <link name="camera_link">
-    <collision>
-      <origin xyz="0.005 0.011 0.013" rpy="0 0 0"/>
-      <geometry>
-        <box size="0.015 0.030 0.027"/>
-      </geometry>
-    </collision>
-  </link>
-  <joint name="camera_rgb_joint" type="fixed">
-    <origin xyz="0.003 0.011 0.009" rpy="0 0 0"/>
-    <parent link="camera_link"/>
-    <child link="camera_rgb_frame"/>
-  </joint>
-  <link name="camera_rgb_frame"/>
-  <joint name="camera_rgb_optical_joint" type="fixed">
-    <origin xyz="0 0 0" rpy="-1.57 0 -1.57"/>
-    <parent link="camera_rgb_frame"/>
-    <child link="camera_rgb_optical_frame"/>
-  </joint>
-  <link name="camera_rgb_optical_frame"/>
 </robot>

File: catkin_ws/src/auefinals/aue_finals/urdf/original/turtlebot3_burger.urdf.xacro (robot description, xacro)
@@ -1,6 +1,6 @@
 <?xml version="1.0" ?>
 <robot name="turtlebot3_burger" xmlns:xacro="http://ros.org/wiki/xacro">
-  <xacro:include filename="$(find finalProject)/urdf/aprilTag/common_properties.xacro"/>
-  <xacro:include filename="$(find finalProject)/urdf/aprilTag/turtlebot3_burger.gazebo.xacro"/>
+  <xacro:include filename="$(find aue_finals)/urdf/original/common_properties.xacro"/>
+  <xacro:include filename="$(find aue_finals)/urdf/original/turtlebot3_burger.gazebo.xacro"/>
   <link name="base_footprint"/>
   <joint name="base_joint" type="fixed">
@@ -140,3 +140,28 @@
     </inertial>
   </link>
+  <joint name="camera_joint" type="fixed">
+    <origin xyz="0.073 -0.011 0.084" rpy="0 0 0"/>
+    <parent link="base_link"/>
+    <child link="camera_link"/>
+  </joint>
+  <link name="camera_link">
+    <collision>
+      <origin xyz="0.005 0.011 0.013" rpy="0 0 0"/>
+      <geometry>
+        <box size="0.015 0.030 0.027"/>
+      </geometry>
+    </collision>
+  </link>
+  <joint name="camera_rgb_joint" type="fixed">
+    <origin xyz="0.003 0.011 0.009" rpy="0 0 0"/>
+    <parent link="camera_link"/>
+    <child link="camera_rgb_frame"/>
+  </joint>
+  <link name="camera_rgb_frame"/>
+  <joint name="camera_rgb_optical_joint" type="fixed">
+    <origin xyz="0 0 0" rpy="-1.57 0 -1.57"/>
+    <parent link="camera_rgb_frame"/>
+    <child link="camera_rgb_optical_frame"/>
+  </joint>
+  <link name="camera_rgb_optical_frame"/>
 </robot>
