Commit message: setup backbone for keyboard implementation, need to fill in if statements

File: catkin_ws/src/auefinals/aue_finals/urdf/aprilTag_robot/turtlebot3_burger.gazebo.xacro (robot description, xacro)
@@ -7,6 +7,6 @@
     <material>Gazebo/DarkGrey</material>
   </gazebo>
-  <gazebo reference="aprilTag_link">
-    <!--material>
+  <!--gazebo reference="aprilTag_link">
+    <material>
       <script>
          <uri>model://aprilTag/materials/scripts</uri>
@@ -14,5 +14,8 @@
          <name>aprilTag</name>
       </script>
-    </material-->
+    </material>
+    <material>aprilTag</material>
+  </gazebo-->
+  <gazebo reference="aprilTag_link">
     <material>aprilTag</material>
   </gazebo>
