Commit message: finished full gazebo implementation for all tasks

File: catkin_ws/src/auefinals/aue_finals/urdf/original/turtlebot3_burger.urdf.xacro (robot description, xacro)
@@ -141,5 +141,5 @@
   </link>
   <joint name="camera_joint" type="fixed">
-    <origin xyz="0.073 -0.011 0.084" rpy="0 0 0"/>
+    <origin xyz="0.073 -0.011 0.084" rpy="0 .15 0"/>
     <parent link="base_link"/>
     <child link="camera_link"/>
